File: Supply and arduino board/My Arduino and supply board/Arduino and supply board/Arduino and supply board.sch (KiCad schematic (older format))
At the start: 5 parts

Commit message: work on my arduino and supply board
Parts:
- removed U?: ATmega328P-PU, Package_DIP:DIP-28_W7.62mm, symbol MCU_Microchip_ATmega:ATmega328P-PU
- added C4, C5, C6: 100n, symbol Device:C
- added GREEN_ON, RX_YELLOW, TX_YELLOW, YELLOW: LED, symbol Device:LED
- added ISCP, ISCP1: ISCP, symbol Connector_Generic:Conn_02x03_Odd_Even
- added POWER: Conn_01x06, symbol Connector_Generic:Conn_01x06
- added R2: 1M, symbol Device:R
- added RESET: SW_MEC_5E, symbol Switch:SW_MEC_5E
- added RESET-EN, UBOOT: SolderJumper_2_Bridged, symbol Jumper:SolderJumper_2_Bridged
- added RN1C, RN1D: 10K, symbol Device:R
- added RN2A, RN2B, RN2C, RN2D, RN4A, RN4B, RN4C, RN4D: 1K, symbol Device:R
- added Y2: 16MHz, symbol Device:Resonator
- added ZIC1: ATmega328P-PU, Package_DIP:DIP-28_W7.62mm, symbol Arduino~and~supply~board-cache:ATmega328P-PU
- U3: renamed from U?; symbol MCU_Microchip_ATmega:ATmega8U2-MU -> Arduino~and~supply~board-cache:MCU_Microchip_ATmega_ATmega8U2-MU
Connections:
- net labels added: +3V3, +5V, AD0, AD1, AD2, AD3, AD4, AD5, AREF, DTR, GND, IO0, IO1, IO2, IO3, IO4, IO5, IO6, IO7, M8RXD, M8TXD, MISO, MISO2, MOSI2, RESET, RESET2, RXLED, SCK, SCK2, TXLED, VIN, XTAL1, XTAL2
- wire segments 6 -> 169
Other:
- moved on the sheet: IOH, J?

Commit message: work on my arduino and supply board
Parts:
- removed U3: ATmega8U2-MU, Package_DFN_QFN:QFN-32-1EP_5x5mm_P0.5mm_EP3.1x3.1mm, symbol Arduino~and~supply~board-cache:MCU_Microchip_ATmega_ATmega8U2-MU
- added C7: 100n, symbol Device:C
- added C8: 1u, symbol Device:C
- added GROUND: SolderJumper_2_Bridged, symbol Jumper:SolderJumper_2_Bridged
- added R1: 1M, symbol Device:R
- added R3: 27R, symbol Device:R
- added U: ATmega16U2-MU, Package_DFN_QFN:QFN-32-1EP_5x5mm_P0.5mm_EP3.1x3.1mm, symbol Arduino~and~supply~board-cache:ATmega16U2-MU
- added Y1: 16MHz, symbol Device:Resonator
Connections:
- net labels added: UGND, USBVCC, VUCAP
- wire segments 169 -> 201
Changed lines of the file:
@@
 $EndDescr
-$Comp
-L Arduino~and~supply~board-cache:MCU_Microchip_ATmega_ATmega8U2-MU U3
-U 1 1 6561175D
-P 3250 3200
-F 0 "U3" H 2650 4550 50  0000 C CNN
-F 1 "ATmega8U2-MU" H 3250 1850 50  0000 C CNN
-F 2 "Package_DFN_QFN:QFN-32-1EP_5x5mm_P0.5mm_EP3.1x3.1mm" H 3250 3200 50  0001 C CIN
-F 3 "http://ww1.microchip.com/downloads/en/DeviceDoc/doc7799.pdf" H 3250 3200 50  0001 C CNN
-	1    3250 3200
-	1    0    0    -1
-$EndComp
 $Comp
 L Connector_Generic:Conn_01x08 IOH
@@
 $EndComp
 Connection ~ 1900 1300
+$Comp
+L Arduino~and~supply~board-cache:ATmega16U2-MU U
+U 1 1 65693AF2
+P 3250 3200
+F 0 "U" H 3250 4667 50  0000 C CNN
+F 1 "ATmega16U2-MU" H 3250 4576 50  0000 C CNN
+F 2 "Package_DFN_QFN:QFN-32-1EP_5x5mm_P0.5mm_EP3.1x3.1mm" H 3250 2200 50  0001 C CIN
+F 3 "http://ww1.microchip.com/downloads/en/DeviceDoc/doc7799.pdf" H 3250 3200 50  0001 C CNN
+	1    3250 3200
+	1    0    0    -1
+$EndComp
+$Comp
+L Device:Resonator Y1
+U 1 1 656C0313
+P 2000 2500
+F 0 "Y1" V 1800 2400 50  0000 L CNN
+F 1 "16MHz" V 2200 2400 50  0000 L CNN
+F 2 "" H 1975 2500 50  0001 C CNN
+F 3 "~" H 1975 2500 50  0001 C CNN
+	1    2000 2500
+	0    1    1    0
+$EndComp
+$Comp
+L Device:R R3
+U 1 1 656C17C4
+P 2300 2650
+F 0 "R3" H 2370 2696 50  0000 L CNN
+F 1 "27R" H 2370 2605 50  0000 L CNN
+F 2 "" V 2230 2650 50  0001 C CNN
+F 3 "~" H 2300 2650 50  0001 C CNN
+	1    2300 2650
+	0    1    1    0
+$EndComp
+$Comp
+L Device:R R1
+U 1 1 656C293A
+P 1450 2500
+F 0 "R1" H 1520 2546 50  0000 L CNN
+F 1 "1M" H 1520 2455 50  0000 L CNN
+F 2 "" V 1380 2500 50  0001 C CNN
+F 3 "~" H 1450 2500 50  0001 C CNN
+	1    1450 2500
+	-1   0    0    1
+$EndComp
+Wire Wire Line
+	2550 2400 2250 2400
+Wire Wire Line
+	2250 2400 2250 2350
+Wire Wire Line
+	2250 2350 2000 2350
+Wire Wire Line
+	2000 2650 2150 2650
+Wire Wire Line
+	2450 2650 2500 2650
+Wire Wire Line
+	2500 2650 2500 2550
+Wire Wire Line
+	2500 2550 2550 2550
+Wire Wire Line
+	1450 2650 2000 2650
+Connection ~ 2000 2650
+Wire Wire Line
+	1450 2350 2000 2350
+Connection ~ 2000 2350
+$Comp
+L power:GND #PWR?
+U 1 1 656F987B
+P 1650 2500
+F 0 "#PWR?" H 1650 2250 50  0001 C CNN
+F 1 "GND" H 1655 2327 50  0000 C CNN
+F 2 "" H 1650 2500 50  0001 C CNN
+F 3 "" H 1650 2500 50  0001 C CNN
+	1    1650 2500
+	1    0    0    -1
+$EndComp
+Wire Wire Line
+	1650 2500 1800 2500
+$Comp
+L Jumper:SolderJumper_2_Bridged GROUND
+U 1 1 65705B3D
+P 2150 4350
+F 0 "GROUND" H 2150 4463 50  0000 C CNN
+F 1 "SolderJumper_2_Bridged" H 2150 4464 50  0001 C CNN
+F 2 "" H 2150 4350 50  0001 C CNN
+F 3 "~" H 2150 4350 50  0001 C CNN
+	1    2150 4350
+	1    0    0    -1
+$EndComp
+$Comp
+L Device:C C8
+U 1 1 65706AC5
+P 1500 4300
+F 0 "C8" H 1615 4346 50  0000 L CNN
+F 1 "1u" H 1615 4255 50  0000 L CNN
+F 2 "" H 1538 4150 50  0001 C CNN
+F 3 "~" H 1500 4300 50  0001 C CNN
+	1    1500 4300
+	1    0    0    -1
+$EndComp
+$Comp
+L Device:C C7
+U 1 1 6570739F
+P 1100 4100
+F 0 "C7" H 1215 4146 50  0000 L CNN
+F 1 "100n" H 1215 4055 50  0000 L CNN
+F 2 "" H 1138 3950 50  0001 C CNN
+F 3 "~" H 1100 4100 50  0001 C CNN
+	1    1100 4100
+	1    0    0    -1
+$EndComp
+Wire Wire Line
+	1500 4150 1500 3650
+Wire Wire Line
+	1500 3650 2550 3650
+Wire Wire Line
+	2550 4350 2400 4350
+Wire Wire Line
+	2000 4350 1950 4350
+Wire Wire Line
+	1950 4350 1950 4650
+Wire Wire Line
+	1950 4650 1500 4650
+Wire Wire Line
+	1500 4650 1500 4450
+$Comp
+L power:GND #PWR?
+U 1 1 6572C936
+P 2400 4350
+F 0 "#PWR?" H 2400 4100 50  0001 C CNN
+F 1 "GND" H 2405 4177 50  0000 C CNN
+F 2 "" H 2400 4350 50  0001 C CNN
+F 3 "" H 2400 4350 50  0001 C CNN
+	1    2400 4350
+	1    0    0    -1
+$EndComp
+Connection ~ 2400 4350
+Wire Wire Line
+	2400 4350 2300 4350
+Text Label 2100 3650 0    50   ~ 0
+VUCAP
+Wire Wire Line
+	1950 4350 1950 4050
+Wire Wire Line
+	1950 4050 2550 4050
+Connection ~ 1950 4350
+Wire Wire Line
+	2400 4350 2400 3300
+Wire Wire Line
+	2400 3300 2550 3300
+Text Label 2100 4050 0    50   ~ 0
+UGND
+Wire Wire Line
+	2550 3750 2100 3750
+Text Label 2100 3750 0    50   ~ 0
+USBVCC
+Wire Wire Line
+	2550 3200 2350 3200
+Wire Wire Line
+	1100 3200 1100 3950
+$Comp
+L power:GND #PWR?
+U 1 1 657638CB
+P 1100 4250
+F 0 "#PWR?" H 1100 4000 50  0001 C CNN
+F 1 "GND" H 1105 4077 50  0000 C CNN
+F 2 "" H 1100 4250 50  0001 C CNN
+F 3 "" H 1100 4250 50  0001 C CNN
+	1    1100 4250
+	1    0    0    -1
+$EndComp
+$Comp
+L power:+5V #PWR?
+U 1 1 65763EDD
+P 2100 3050
+F 0 "#PWR?" H 2100 2900 50  0001 C CNN
+F 1 "+5V" H 2115 3223 50  0000 C CNN
+F 2 "" H 2100 3050 50  0001 C CNN
+F 3 "" H 2100 3050 50  0001 C CNN
+	1    2100 3050
+	1    0    0    -1
+$EndComp
+Wire Wire Line
+	2550 2850 2450 2850
+Wire Wire Line
+	2450 2850 2450 3100
+Wire Wire Line
+	2450 3100 2350 3100
+Wire Wire Line
+	2100 3100 2100 3050
+Wire Wire Line
+	2350 3200 2350 3100
+Connection ~ 2350 3200
+Wire Wire Line
+	2350 3200 1100 3200
+Connection ~ 2350 3100
+Wire Wire Line
+	2350 3100 2100 3100
 $EndSCHEMATC

Commit message: new work on Arduino and supply board
Parts:
- added C10, C11, C12, C9: 22p, symbol Device:C
- added F1: 500mA, symbol Device:Fuse
- added L1: BLM21, symbol Device:L
- added Q1, Q2: 16MHz, symbol Device:Crystal
- added RN3D, RND3A: 22R, symbol Device:R
- added X1: USB_B, symbol Connector:USB_B
- added Z1, Z2: PGB1010604, symbol Device:Varistor
- renumbered U to U3
Connections:
- net labels added: D+, D-, RD+, RD-, USHIELD, XT1, XT2, XUSB
- wire segments 201 -> 246
Other:
- moved on the sheet: C4, C5, C6, C7, C8, GREEN_ON, GROUND, IOH, ISCP, ISCP1, J?, POWER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

Commit message: work on arduino board, every components have package
Parts:
- added C1, C2: 100n, Capacitor_SMD:C_0603_1608Metric, symbol Device:C
- added C3: 1u, Capacitor_SMD:C_0603_1608Metric, symbol Device:C
- added D1: M7, Diode_SMD:D_SMB, symbol Device:D
- added IC1: MC33269ST-5.0T3, Package_TO_SOT_SMD:SOT-223, symbol Arduino~and~supply~board-cache:MC33269ST-5.0T3
- added IC2: MC33269D-5.0, Package_TO_SOT_SMD:SOT-223-3_TabPin2, symbol Arduino~and~supply~board-cache:MC33269D-5.0
- added J1: Barrel_Jack_MountingPin, Connector_BarrelJack:BarrelJack_Horizontal, symbol Arduino~and~supply~board-cache:Connector_Barrel_Jack_MountingPin
- added PC1, PC2: 47u, Capacitor_SMD:CP_Elec_6.3x9.9, symbol Device:CP
- added RN1A1, RN1B1: 10K, Resistor_SMD:R_0402_1005Metric, symbol Device:R
- added T1: FDN340V, Package_TO_SOT_SMD:SOT-23, symbol Transistor_FET:FDN340P
- added U1: LP2985-3.3, Package_TO_SOT_SMD:SOT-23-5_HandSoldering, symbol Arduino~and~supply~board-cache:LP2985-3.3
- added U1A1, U1B1, U1C1: LM358D, Package_SO:MSOP-8_3x3mm_P0.65mm, symbol Arduino~and~supply~board-cache:LM358
- AD1: renamed from J?; footprint (none) -> Connector_PinHeader_2.54mm:PinHeader_1x06_P2.54mm_Vertical
- C10, C11, C12, C4, C5, C6, C7, C8, C9: footprint (none) -> Capacitor_SMD:C_0603_1608Metric
- F1: footprint (none) -> Resistor_SMD:R_1812_4532Metric
- GREEN_ON1: renamed from GREEN_ON; footprint (none) -> LED_SMD:LED_0805_2012Metric
- GROUND1: renamed from GROUND; footprint (none) -> Jumper:SolderJumper-2_P1.3mm_Bridged_Pad1.0x1.5mm
- IOH1: renamed from IOH; footprint (none) -> Connector_PinHeader_2.54mm:PinHeader_1x08_P2.54mm_Vertical
- IOL1: renamed from J?; footprint (none) -> Connector_PinHeader_2.54mm:PinHeader_1x08_P2.54mm_Vertical
- ISCP1: footprint (none) -> Connector_PinHeader_2.54mm:PinHeader_2x03_P2.54mm_Vertical
- ISCP2: renamed from ISCP; footprint (none) -> Connector_PinHeader_2.54mm:PinHeader_2x03_P2.54mm_Vertical
- L1: footprint (none) -> Inductor_SMD:L_0805_2012Metric
- POWER1: renamed from POWER; footprint (none) -> Connector_PinHeader_2.54mm:PinHeader_1x06_P2.54mm_Vertical
- Q1, Q2: footprint (none) -> Crystal:Crystal_HC18-U_Vertical
- R1, R2, R3: footprint (none) -> Resistor_SMD:R_0402_1005Metric
- RESET-EN1: renamed from RESET-EN; footprint (none) -> Jumper:SolderJumper-2_P1.3mm_Bridged_Pad1.0x1.5mm
- RESET1: renamed from RESET; footprint (none) -> Button_Switch_SMD:SW_DIP_SPSTx02_Slide_6.7x6.64mm_W6.73mm_P2.54mm_LowProfile_JPin
- RN1C1: renamed from RN1C; footprint (none) -> Resistor_SMD:R_0402_1005Metric
- RN1D1: renamed from RN1D; footprint (none) -> Resistor_SMD:R_0402_1005Metric
- RN2A1: renamed from RN2A; footprint (none) -> Resistor_SMD:R_0402_1005Metric
- RN2B1: renamed from RN2B; footprint (none) -> Resistor_SMD:R_0402_1005Metric
- RN2C1: renamed from RN2C; footprint (none) -> Resistor_SMD:R_0402_1005Metric
- RN2D1: renamed from RN2D; footprint (none) -> Resistor_SMD:R_0402_1005Metric
- RN3D1: renamed from RN3D; footprint (none) -> Resistor_SMD:R_0402_1005Metric
- RN4A1: renamed from RN4A; footprint (none) -> Resistor_SMD:R_0402_1005Metric
- RN4B1: renamed from RN4B; footprint (none) -> Resistor_SMD:R_0402_1005Metric
- RN4C1: renamed from RN4C; footprint (none) -> Resistor_SMD:R_0402_1005Metric
- RN4D1: renamed from RN4D; footprint (none) -> Resistor_SMD:R_0402_1005Metric
- RND3A1: renamed from RND3A; footprint (none) -> Resistor_SMD:R_0402_1005Metric
- RX_YELLOW1: renamed from RX_YELLOW; footprint (none) -> LED_SMD:LED_0805_2012Metric
- TX_YELLOW1: renamed from TX_YELLOW; footprint (none) -> LED_SMD:LED_0805_2012Metric
- UBOOT1: renamed from UBOOT; footprint (none) -> Jumper:SolderJumper-2_P1.3mm_Bridged_Pad1.0x1.5mm
- X1: footprint (none) -> Connector_USB:USB_Mini-B_Wuerth_65100516121_Horizontal
- Y1, Y2: footprint (none) -> Crystal:Resonator_SMD-3Pin_7.2x3.0mm
- YELLOW1: renamed from YELLOW; footprint (none) -> LED_SMD:LED_0805_2012Metric
- Z1, Z2: footprint (none) -> Resistor_SMD:R_0603_1608Metric
Connections:
- net labels added: CMP, GATE_CMD, PWRIM
- wire segments 246 -> 301

Commit message: new work on arduino board
Parts:
- removed IC1: MC33269ST-5.0T3, Package_TO_SOT_SMD:SOT-223, symbol Arduino~and~supply~board-cache:MC33269ST-5.0T3
- removed IC2: MC33269D-5.0, Package_TO_SOT_SMD:SOT-223-3_TabPin2, symbol Arduino~and~supply~board-cache:MC33269D-5.0
- removed J1: Barrel_Jack_MountingPin, Connector_BarrelJack:BarrelJack_Horizontal, symbol Arduino~and~supply~board-cache:Connector_Barrel_Jack_MountingPin
- added Conn1: Connector_Barrel_Jack_MountingPin-Arduino_and_sup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, Connector_BarrelJack:BarrelJack_Horizontal, symbol Arduino-and-supply-board-rescue:Connector_Barrel_Jack_MountingPin-Arduino_and_s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
- added IC1: MC33269ST-5.0T3-Arduino_and_supply_board-cache, Package_TO_SOT_SMD:SOT-223, symbol Arduino-and-supply-board-rescue:MC33269ST-5.0T3-Arduino_and_supply_board-cache
- added IC2: MC33269D-5.0-Arduino_and_supply_board-cache, Package_TO_SOT_SMD:SOT-223-3_TabPin2, symbol Arduino-and-supply-board-rescue:MC33269D-5.0-Arduino_and_supply_board-cache
Changed lines of the file:
@@
 VIN
-$Comp
-L Arduino~and~supply~board-cache:Connector_Barrel_Jack_MountingPin J1
-U 1 1 658435F4
-P 9100 1650
-F 0 "J1" H 9157 1967 50  0000 C CNN
-F 1 "Barrel_Jack_MountingPin" H 9157 1876 50  0001 C CNN
-F 2 "Connector_BarrelJack:BarrelJack_Horizontal" H 9150 1610 50  0001 C CNN
-F 3 "~" H 9150 1610 50  0001 C CNN
-	1    9100 1650
-	1    0    0    -1
-$EndComp
 $Comp
 L Device:D D1
@@
 $EndComp
 $Comp
-L Arduino~and~supply~board-cache:MC33269ST-5.0T3 IC1
-U 1 1 657E56D9
-P 11250 1050
-F 0 "IC1" H 11250 1392 50  0000 C CNN
-F 1 "MC33269ST-5.0T3" H 11250 1301 50  0000 C CNN
-F 2 "Package_TO_SOT_SMD:SOT-223" H 11250 1100 50  0001 C CNN
-F 3 "" H 11250 1100 50  0001 C CNN
-	1    11250 1050
-	1    0    0    -1
-$EndComp
-$Comp
 L power:+5V #PWR0130
 U 1 1 65806B0F
@@
 VIN
 $Comp
-L Arduino~and~supply~board-cache:MC33269D-5.0 IC2
-U 1 1 659797E7
+L Arduino-and-supply-board-rescue:MC33269D-5.0-Arduino_and_supply_board-cache IC2
+U 1 1 6571603C
 P 11200 1850
 F 0 "IC2" H 11200 2092 50  0000 C CNN
-F 1 "MC33269D-5.0" H 11200 2001 50  0000 C CNN
+F 1 "MC33269D-5.0-Arduino_and_supply_board-cache" H 11200 2001 50  0000 C CNN
 F 2 "Package_TO_SOT_SMD:SOT-223-3_TabPin2" H 11225 1700 50  0001 L CIN
 F 3 "" H 11200 1800 50  0001 C CNN
@@
 	1    0    0    -1
 $EndComp
+$Comp
+L Arduino-and-supply-board-rescue:MC33269ST-5.0T3-Arduino_and_supply_board-cache IC1
+U 1 1 65716E1B
+P 11250 1050
+F 0 "IC1" H 11250 1392 50  0000 C CNN
+F 1 "MC33269ST-5.0T3-Arduino_and_supply_board-cache" H 11250 1301 50  0000 C CNN
+F 2 "Package_TO_SOT_SMD:SOT-223" H 11250 1100 50  0001 C CNN
+F 3 "" H 11250 1100 50  0001 C CNN
+	1    11250 1050
+	1    0    0    -1
+$EndComp
+$Comp
+L Arduino-and-supply-board-rescue:Connector_Barrel_Jack_MountingPin-Arduino_and_supply_board-cache Conn1
+U 1 1 65719DC7
+P 9100 1650
+F 0 "Conn1" H 9157 1967 50  0000 C CNN
+F 1 "Connector_Barrel_Jack_MountingPin-Arduino_and_supply_board-cache" H 9157 1876 50  0000 C CNN
+F 2 "Connector_BarrelJack:BarrelJack_Horizontal" H 9150 1610 50  0001 C CNN
+F 3 "" H 9150 1610 50  0001 C CNN
+	1    9100 1650
+	1    0    0    -1
+$EndComp

Commit message: every part on board is connected
Parts:
- added Cboot1, Cinx1: 100n, Capacitor_SMD:C_0603_1608Metric, symbol Device:C
- added Cff1: 47p, Capacitor_SMD:C_0603_1608Metric, symbol Device:C
- added Cin1: 10u, Capacitor_SMD:C_0603_1608Metric, symbol Device:C
- added Cout1: 47u, Capacitor_SMD:C_0603_1608Metric, symbol Device:C
- added Css1: 33n, Capacitor_SMD:C_0603_1608Metric, symbol Device:C
- added L2: 15u, Inductor_SMD:L_Taiyo-Yuden_MD-5050, symbol Device:L
- added Rfbb1: 10K, Resistor_SMD:R_0402_1005Metric, symbol Device:R
- added Rfbt1: 140K, Resistor_SMD:R_0402_1005Metric, symbol Device:R
- added U4: TPS629DRL, Package_TO_SOT_SMD:TSOT-23-8, symbol Arduino~and~supply~board-cache:Arduino_and_supply_board-cache_TPS629DRL
- added Vin1, Vout1: Conn_01x02, Connector_PinSocket_2.54mm:PinSocket_1x02_P2.54mm_Vertical, symbol Connector_Generic:Conn_01x02
- U3: symbol Arduino~and~supply~board-cache:ATmega16U2-MU -> Arduino~and~supply~board-cache:Arduino_and_supply_board-cache_ATmega16U2-MU
Connections:
- wire segments 301 -> 335
Other:
- moved on the sheet: C2, Conn1, D1, IC1, IC2, PC1, PC2

Commit message: new work on board
Parts:
- removed U4: TPS629DRL, Package_TO_SOT_SMD:TSOT-23-8, symbol Arduino~and~supply~board-cache:Arduino_and_supply_board-cache_TPS629DRL
- added U4: Arduino_and_supply_board-cache_Arduino_and_supply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, Package_TO_SOT_SMD:TSOT-23-8, symbol Arduino~and~supply~board-cache:Arduino_and_supply_board-cache_Arduino_and_suppl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
- U3: symbol Arduino~and~supply~board-cache:Arduino_and_supply_board-cache_ATmega16U2-MU -> Arduino-and-supply-board-rescue:Arduino_and_supply_board-cache_ATmega16U2-MU-Arduino~and~supply~board-cache
Changed lines of the file:
@@
 Connection ~ 4500 4600
 $Comp
-L Arduino~and~supply~board-cache:Arduino_and_supply_board-cache_ATmega16U2-MU U3
+L Arduino-and-supply-board-rescue:Arduino_and_supply_board-cache_ATmega16U2-MU-Arduino~and~supply~board-cache U3
 U 1 1 65693AF2
 P 5850 6500
@@
 $EndComp
 $Comp
-L Arduino~and~supply~board-cache:Arduino_and_supply_board-cache_TPS629DRL U4
-U 1 1 6572413E
-P 13100 1500
-F 0 "U4" H 13000 1875 50  0000 C CNN
-F 1 "TPS629DRL" H 13000 1784 50  0000 C CNN
-F 2 "Package_TO_SOT_SMD:TSOT-23-8" H 13100 1500 50  0001 C CNN
-F 3 "" H 13100 1500 50  0001 C CNN
-	1    13100 1500
-	1    0    0    -1
-$EndComp
-$Comp
 L Device:C Css1
 U 1 1 65724CD8
@@
 	1    0    0    -1
 $EndComp
+$Comp
+L Arduino~and~supply~board-cache:Arduino_and_supply_board-cache_Arduino_and_supply_board-cache_TPS629DRL U4
+U 1 1 65732BE4
+P 13100 1500
+F 0 "U4" H 13000 1875 50  0000 C CNN
+F 1 "Arduino_and_supply_board-cache_Arduino_and_supply_board-cache_TPS629DRL" H 13000 1784 50  0000 C CNN
+F 2 "Package_TO_SOT_SMD:TSOT-23-8" H 13100 1500 50  0001 C CNN
+F 3 "" H 13100 1500 50  0001 C CNN
+	1    13100 1500
+	1    0    0    -1
+$EndComp

Commit message: big changes on arduino board
Parts:
- removed AD1: Conn_01x06, Connector_PinHeader_2.54mm:PinHeader_1x06_P2.54mm_Vertical, symbol Connector_Generic:Conn_01x06
- removed C11: 22p, Capacitor_SMD:C_0603_1608Metric, symbol Device:C
- removed Conn1: Connector_Barrel_Jack_MountingPin-Arduino_and_sup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, Connector_BarrelJack:BarrelJack_Horizontal, symbol Arduino-and-supply-board-rescue:Connector_Barrel_Jack_MountingPin-Arduino_and_s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
- removed F1: 500mA, Resistor_SMD:R_1812_4532Metric, symbol Device:Fuse
- removed GROUND1, RESET-EN1, UBOOT1: SolderJumper_2_Bridged, Jumper:SolderJumper-2_P1.3mm_Bridged_Pad1.0x1.5mm, symbol Jumper:SolderJumper_2_Bridged
- removed IC1: MC33269ST-5.0T3-Arduino_and_supply_board-cache, Package_TO_SOT_SMD:SOT-223, symbol Arduino-and-supply-board-rescue:MC33269ST-5.0T3-Arduino_and_supply_board-cache
- removed IC2: MC33269D-5.0-Arduino_and_supply_board-cache, Package_TO_SOT_SMD:SOT-223-3_TabPin2, symbol Arduino-and-supply-board-rescue:MC33269D-5.0-Arduino_and_supply_board-cache
- removed IOH1, IOL1: Conn_01x08, Connector_PinHeader_2.54mm:PinHeader_1x08_P2.54mm_Vertical, symbol Connector_Generic:Conn_01x08
- removed ISCP1, ISCP2: ISCP, Connector_PinHeader_2.54mm:PinHeader_2x03_P2.54mm_Vertical, symbol Connector_Generic:Conn_02x03_Odd_Even
- removed L1: BLM21, Inductor_SMD:L_0805_2012Metric, symbol Device:L
- removed Q1: 16MHz, Crystal:Crystal_HC18-U_Vertical, symbol Device:Crystal
- removed RN1C1: 10K, Resistor_SMD:R_0402_1005Metric, symbol Device:R
- removed RN2A1, RN2B1, RN4C1: 1K, Resistor_SMD:R_0402_1005Metric, symbol Device:R
- removed RN3D1, RND3A1: 22R, Resistor_SMD:R_0402_1005Metric, symbol Device:R
- removed T1: FDN340V, Package_TO_SOT_SMD:SOT-23, symbol Transistor_FET:FDN340P
- removed U1: LP2985-3.3, Package_TO_SOT_SMD:SOT-23-5_HandSoldering, symbol Arduino~and~supply~board-cache:LP2985-3.3
- removed U1A1, U1B1, U1C1: LM358D, Package_SO:MSOP-8_3x3mm_P0.65mm, symbol Arduino~and~supply~board-cache:LM358
- removed U3: ATmega16U2-MU, Package_DFN_QFN:QFN-32-1EP_5x5mm_P0.5mm_EP3.1x3.1mm, symbol Arduino-and-supply-board-rescue:Arduino_and_supply_board-cache_ATmega16U2-MU-Ar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
- removed U4: Arduino_and_supply_board-cache_Arduino_and_supply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, Package_TO_SOT_SMD:TSOT-23-8, symbol Arduino~and~supply~board-cache:Arduino_and_supply_board-cache_Arduino_and_suppl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
- removed X1: USB_B, Connector_USB:USB_Mini-B_Wuerth_65100516121_Horizontal, symbol Connector:USB_B
- removed Y1: 16MHz, Crystal:Resonator_SMD-3Pin_7.2x3.0mm, symbol Device:Resonator
- removed YELLOW1: LED, LED_SMD:LED_0805_2012Metric, symbol Device:LED
- removed Z1, Z2: PGB1010604, Resistor_SMD:R_0603_1608Metric, symbol Device:Varistor
- removed ZIC1: ATmega328P-PU, Package_DIP:DIP-28_W7.62mm, symbol Arduino~and~supply~board-cache:ATmega328P-PU
- added FB1: Ferrite_Bead, Resistor_SMD:R_0603_1608Metric, symbol Device:Ferrite_Bead
- added J1: USB_C_Receptacle_USB2.0, Connector_USB:USB_C_Receptacle_HRO_TYPE-C-31-M-12, symbol Connector:USB_C_Receptacle_USB2.0
- added J2, J3, J4, J5, J6, J7: Conn_01x03, Connector_PinSocket_2.54mm:PinSocket_1x03_P2.54mm_Vertical, symbol Connector_Generic:Conn_01x03
- added T1: FDN340V, Package_TO_SOT_SMD:SOT-23, symbol Assembly_board_schem:FDN340V
- added U1: LM358D, Package_SO:MSOP-8_3x3mm_P0.65mm, symbol Assembly_board_schem:LM358D
- added U2: LP2985-3.3, Package_TO_SOT_SMD:SOT-23-5_HandSoldering, symbol Assembly_board_schem:LP2985-3.3
- added U3: MC33269D-5.0, Package_TO_SOT_SMD:SOT-223-3_TabPin2, symbol Assembly_board_schem:MC33269D-5.0
- added U4: MC33269ST-5.0T3, Package_TO_SOT_SMD:SOT-223, symbol Assembly_board_schem:MC33269ST-5.0T3
- added U5: TPS629DRL, Package_TO_SOT_SMD:TSOT-23-8, symbol Assembly_board_schem:TPS629DRL
- added U7: Atmega328P-PU, Package_QFP:TQFP-32_7x7mm_P0.8mm, symbol Assembly_board_schem:Atmega328P-PU
- added U8: FT231XQ, Package_DFN_QFN:QFN-20-1EP_4x4mm_P0.5mm_EP2.5x2.5mm, symbol Assembly_board_schem:FT231XQ
- added Vin2: Conn_01x02, Connector_PinSocket_2.54mm:PinSocket_1x02_P2.54mm_Vertical, symbol Connector_Generic:Conn_01x02
- C5: value 100n -> 10n
- C7: value 100n -> 47p
- C8: value 1u -> 47p
- C9: value 22p -> 100n
- R1: value 1M -> 27R
- renumbered Cin1 to C13, Cinx1 to C14, Css1 to C15, Cboot1 to C16, Cff1 to C17, Cout1 to C18, RN2C1 to R10, RN1D1 to R11, RN4B1 to R12, RN4A1 to R13, RN4D1 to R16, Rfbt1 to R18, Rfbb1 to R19, RN1B1 to R4, RN1A1 to R5, RN2D1 to R9
Connections:
- net labels removed: D+, D-, DTR, IO0, IO1, IO2, IO3, IO4, IO5, IO6, IO7, IO8, IO9, MISO, MISO2, MOSI, MOSI2, RD+, RD-, RESET2, SCK, SCK2, SS, UGND, USHIELD, VUCAP, XT1, XT2, XUSB
- wire segments 335 -> 241
Other:
- moved on the sheet: C4, R10, R9, RESET1, RX_YELLOW1, TX_YELLOW1
